File: crt.sch (KiCad schematic (older format))
At the start: 121 parts, among them J1 Video, J2 H_COIL, J3 V_COIL, J4 CRT, J5 Barrel_Jack, Q1 BC847, Q2 2N5551, Q3 9013, Q4 9013, Q5 NPN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

Commit message: fix munting pads, camera ready?
Parts:
- added H1, H2, H3, H4: MountingHole_Pad, MountingHole:MountingHole_3.2mm_M3_Pad_Via, symbol Mechanical:MountingHole_Pad
Connections:
- net GND: now also H1.1, H2.1, H3.1, H4.1
Changed lines of the file:
@@
 Wire Wire Line
 	3300 9150 3550 9150
+$Comp
+L Mechanical:MountingHole_Pad H1
+U 1 1 5FAAFBF3
+P 7250 10350
+F 0 "H1" H 7350 10353 50  0000 L CNN
+F 1 "MountingHole_Pad" H 7350 10308 50  0001 L CNN
+F 2 "MountingHole:MountingHole_3.2mm_M3_Pad_Via" H 7250 10350 50  0001 C CNN
+F 3 "~" H 7250 10350 50  0001 C CNN
+	1    7250 10350
+	1    0    0    -1
+$EndComp
+$Comp
+L Mechanical:MountingHole_Pad H2
+U 1 1 5FAB0126
+P 7550 10350
+F 0 "H2" H 7650 10353 50  0000 L CNN
+F 1 "MountingHole_Pad" H 7650 10308 50  0001 L CNN
+F 2 "MountingHole:MountingHole_3.2mm_M3_Pad_Via" H 7550 10350 50  0001 C CNN
+F 3 "~" H 7550 10350 50  0001 C CNN
+	1    7550 10350
+	1    0    0    -1
+$EndComp
+$Comp
+L Mechanical:MountingHole_Pad H3
+U 1 1 5FAD2138
+P 7850 10350
+F 0 "H3" H 7950 10353 50  0000 L CNN
+F 1 "MountingHole_Pad" H 7950 10308 50  0001 L CNN
+F 2 "MountingHole:MountingHole_3.2mm_M3_Pad_Via" H 7850 10350 50  0001 C CNN
+F 3 "~" H 7850 10350 50  0001 C CNN
+	1    7850 10350
+	1    0    0    -1
+$EndComp
+$Comp
+L Mechanical:MountingHole_Pad H4
+U 1 1 5FAD2142
+P 8150 10350
+F 0 "H4" H 8250 10353 50  0000 L CNN
+F 1 "MountingHole_Pad" H 8250 10308 50  0001 L CNN
+F 2 "MountingHole:MountingHole_3.2mm_M3_Pad_Via" H 8150 10350 50  0001 C CNN
+F 3 "~" H 8150 10350 50  0001 C CNN
+	1    8150 10350
+	1    0    0    -1
+$EndComp
+$Comp
+L power:GND #PWR0153
+U 1 1 5FAF44EF
+P 7250 10550
+F 0 "#PWR0153" H 7250 10300 50  0001 C CNN
+F 1 "GND" H 7255 10377 50  0000 C CNN
+F 2 "" H 7250 10550 50  0001 C CNN
+F 3 "" H 7250 10550 50  0001 C CNN
+	1    7250 10550
+	1    0    0    -1
+$EndComp
+Wire Wire Line
+	7250 10550 7250 10500
+Wire Wire Line
+	7250 10500 7550 10500
+Wire Wire Line
+	8150 10500 8150 10450
+Connection ~ 7250 10500
+Wire Wire Line
+	7250 10500 7250 10450
+Wire Wire Line
+	7850 10500 7850 10450
+Connection ~ 7850 10500
+Wire Wire Line
+	7850 10500 8150 10500
+Wire Wire Line
+	7550 10500 7550 10450
+Connection ~ 7550 10500
+Wire Wire Line
+	7550 10500 7850 10500
 $EndSCHEMATC
